Commit message: Fix urdf to keep dh convention

File: RPP.urdf (robot description, URDF)
Before this commit: robot RPP, 5 links, 4 joints
Joints:
- joint Joint3: origin xyz=0 0 0.46 rpy=0 1.57 0 -> xyz=0 0 0.46 rpy=1.57 0 1.57
- joint ee_link: origin xyz=0 0 0.15 rpy=0 0 0 -> xyz=0 0 0.15 rpy=0 0 -1.57

Commit message: Write report for first assignment (kinematics and jacobians)

File: RPP.urdf (robot description, URDF)
Before this commit: robot RPP, 5 links, 4 joints
Joints:
- joint Joint3: origin xyz=0 0 0.46 rpy=1.57 0 1.57 -> xyz=0 0 0.46 rpy=-1.57 0 -1.57
- joint ee_link: origin xyz=0 0 0.15 rpy=0 0 -1.57 -> xyz=0 0 0.15 rpy=0 0 1.57
